File: Continuity_Tester.sch (EAGLE design)
At the start: 12 parts

Commit message: Add files via upload
Parts:
- D1: device lab1:LED -> lab1:DIODE
Changed lines of the file:
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@@
 <part name="J1" library="lab1" deviceset="POWER" device=""/>
 <part name="S1" library="lab1" deviceset="SWITCH" device=""/>
-<part name="D1" library="lab1" deviceset="LED" device=""/>
 <part name="R1" library="lab1" deviceset="RES" device="" value="2k"/>
 <part name="R2" library="lab1" deviceset="RES" device="" value="10k"/>
@@
 <part name="J3" library="lab1" deviceset="ALLIGATORCLIP" device=""/>
 <part name="SUPPLY3" library="lab1" deviceset="GND" device=""/>
+<part name="D1" library="lab1" deviceset="DIODE" device=""/>
 </parts>
 <sheets>
@@
 <instance part="J1" gate="G$1" x="83.82" y="132.08"/>
 <instance part="S1" gate="G$1" x="114.3" y="127" rot="R270"/>
-<instance part="D1" gate="G$1" x="149.86" y="119.38"/>
 <instance part="R1" gate="G$1" x="149.86" y="99.06" rot="R90"/>
 <instance part="R2" gate="G$1" x="170.18" y="99.06" rot="R90"/>
@@
 <instance part="J3" gate="G$1" x="149.86" y="43.18"/>
 <instance part="SUPPLY3" gate="PE" x="170.18" y="20.32"/>
+<instance part="D1" gate="G$1" x="149.86" y="119.38" rot="R270"/>
 </instances>
 <busses>
@@
 <segment>
 <pinref part="S1" gate="G$1" pin="3"/>
-<pinref part="D1" gate="G$1" pin="A"/>
 <wire x1="119.38" y1="127" x2="149.86" y2="127" width="0.1524" layer="91"/>
 <wire x1="149.86" y1="127" x2="149.86" y2="121.92" width="0.1524" layer="91"/>
+<pinref part="D1" gate="G$1" pin="A"/>
 </segment>
 </net>
 <net name="N$3" class="0">
 <segment>
-<pinref part="D1" gate="G$1" pin="C"/>
 <pinref part="R1" gate="G$1" pin="2"/>
-<wire x1="149.86" y1="114.3" x2="149.86" y2="109.22" width="0.1524" layer="91"/>
+<wire x1="149.86" y1="116.84" x2="149.86" y2="109.22" width="0.1524" layer="91"/>
 <wire x1="149.86" y1="109.22" x2="149.86" y2="104.14" width="0.1524" layer="91"/>
 <wire x1="149.86" y1="109.22" x2="170.18" y2="109.22" width="0.1524" layer="91"/>
@@
 <wire x1="219.82" y1="105.52" x2="213.36" y2="109.22" width="0.1524" layer="91"/>
 <junction x="213.36" y="109.22"/>
+<pinref part="D1" gate="G$1" pin="C"/>
 </segment>
 </net>
